Commit message: first upload

File: src/diff_wheeled_robot_gazebo/urdf/diff_wheeled_robot.xacro (robot description, xacro)
@@ -56,4 +56,17 @@
     </inertial>
     <visual>
+    <origin xyz="0.16 0 0" rpy="0 0 0" /> <!-- 车头位于车体中央 -->
+    <geometry>
+      <box size="0.04 0.04 0.04" /> <!-- 小方块尺寸 -->
+    </geometry>
+    <material name="White" />
+  </visual>
+  <collision>
+    <origin xyz="0.16 0 0" rpy="0 0 0 " /> <!-- 与visual的origin对齐 -->
+    <geometry>
+      <box size="0.04 0.04 0.04" />
+    </geometry>
+  </collision>
+    <visual>
       <origin xyz="0 0 0" rpy="0 0 0" />
       <geometry>
