Commit message: add printmap

File: src/differential_4-wheeled_car/urdf/differential_4-wheeled_car.xacro (robot description, xacro)
@@ -1,5 +1,5 @@
 <?xml version="1.0"?>
 <robot name="differential_4-wheeled_car" xmlns:xacro="http://www.ros.org/wiki/xacro">
-  <xacro:include filename="$(find differential_4-wheeled_car)/urdf/wheel.urdf.xacro" />
+  <xacro:include filename="$(find differential_4-wheeled_car)/urdf/wheel.xacro" />
 <!-- Defining the colors used in this robot -->
   <material name="Black">
@@ -110,3 +110,15 @@
     </plugin>
   </gazebo>
+  <gazebo>
+    <plugin name="p3d_base_controller" filename="libgazebo_ros_p3d.so">
+      <alwaysOn>true</alwaysOn>
+      <updateRate>50.0</updateRate>
+      <bodyName>base_link</bodyName>
+      <topicName>base_pose_ground_truth</topicName>
+      <gaussianNoise>0.0</gaussianNoise>
+      <frameName>map</frameName>
+      <xyzOffsets>0 0 0</xyzOffsets>
+      <rpyOffsets>0 0 0</rpyOffsets>
+    </plugin>
+  </gazebo>
 </robot>

File: src/differential_4-wheeled_car/urdf/wheel.xacro (robot description, xacro)
@@ -51,13 +51,4 @@
       <joint_properties damping="0.0" friction="0.0"/>
     </joint>
-    <!-- Transmission is important to link the joints and the controller -->
-    <transmission name="${fb}_${lr}_wheel_joint_trans">
-      <type>transmission_interface/SimpleTransmission</type>
-      <joint name="${fb}_${lr}_wheel_joint" />
-      <actuator name="${fb}_${lr}_wheel_joint_motor">
-        <hardwareInterface>EffortJointInterface</hardwareInterface>
-        <mechanicalReduction>1</mechanicalReduction>
-      </actuator>
-    </transmission>
   </xacro:macro>
 </robot>

Commit message: add lab3

File: src/differential_4-wheeled_car/urdf/differential_4-wheeled_car.xacro (robot description, xacro)
@@ -2,4 +2,6 @@
 <robot name="differential_4-wheeled_car" xmlns:xacro="http://www.ros.org/wiki/xacro">
   <xacro:include filename="$(find differential_4-wheeled_car)/urdf/wheel.xacro" />
+  <xacro:include filename="$(find differential_4-wheeled_car)/urdf/my_sensors_laser.urdf.xacro" />
+  <xacro:include filename="$(find differential_4-wheeled_car)/urdf/my_laser.urdf.xacro" />
 <!-- Defining the colors used in this robot -->
   <material name="Black">
@@ -14,4 +16,7 @@
   <material name="Blue">
     <color rgba="0.0 0.0 0.8 1.0"/>
+  </material>
+  <material name="DarkGray">
+    <color rgba="0.66 0.66 0.66 1.0"/>
   </material>
   <!-- xacro:PROPERTY LIST -->
